Commit message: All works on real robot. Not clearly but works.

File: src/my_robot_moveit_config/config/armassem1.ros2_control.xacro (robot description, xacro)
@@ -1,10 +1,25 @@
 <?xml version="1.0"?>
 <robot xmlns:xacro="http://www.ros.org/wiki/xacro">
-    <xacro:macro name="armassem1_ros2_control" params="name initial_positions_file">
+    <xacro:macro name="armassem1_ros2_control" params="name initial_positions_file use_mock_hardware:=true serial_port:=/dev/ttyACM0 baud_rate:=115200">
         <xacro:property name="initial_positions" value="${xacro.load_yaml(initial_positions_file)['initial_positions']}"/>
+        <xacro:property name="joint1_steps_per_radian" value="${(1600.0 * 18.0) / (2.0 * 3.141592653589793)}"/>
+        <xacro:property name="joint2_steps_per_radian" value="${(800.0 * 80.0) / (2.0 * 3.141592653589793)}"/>
+        <xacro:property name="joint3_steps_per_radian" value="${(800.0 * 80.0) / (2.0 * 3.141592653589793)}"/>
+        <xacro:property name="joint4_steps_per_radian" value="${(800.0 * 50.0) / (2.0 * 3.141592653589793)}"/>
+        <xacro:property name="joint5_steps_per_radian" value="${(800.0 * 30.0) / (2.0 * 3.141592653589793)}"/>
         <ros2_control name="${name}" type="system">
             <hardware>
-                <!-- By default, set up controllers for simulation. This won't work on real hardware -->
-                <plugin>mock_components/GenericSystem</plugin>
+                <xacro:if value="${use_mock_hardware}">
+                    <plugin>mock_components/GenericSystem</plugin>
+                </xacro:if>
+                <xacro:unless value="${use_mock_hardware}">
+                    <plugin>robot_arm_hardware/RobotArmSystem</plugin>
+                    <param name="serial_port">${serial_port}</param>
+                    <param name="baud_rate">${baud_rate}</param>
+                    <param name="command_tolerance_rad">0.0005</param>
+                    <param name="state_poll_period_sec">0.02</param>
+                    <param name="min_command_period_sec">0.005</param>
+                    <param name="min_step_delta_to_resend">1</param>
+                </xacro:unless>
             </hardware>
             <joint name="Joint_1_Joint">
@@ -14,4 +29,5 @@
                 </state_interface>
                 <state_interface name="velocity"/>
+                <param name="steps_per_radian">${joint1_steps_per_radian}</param>
             </joint>
             <joint name="Joint_2_Joint">
@@ -21,4 +37,5 @@
                 </state_interface>
                 <state_interface name="velocity"/>
+                <param name="steps_per_radian">${joint2_steps_per_radian}</param>
             </joint>
             <joint name="Joint_3_Joint">
@@ -28,4 +45,5 @@
                 </state_interface>
                 <state_interface name="velocity"/>
+                <param name="steps_per_radian">${joint3_steps_per_radian}</param>
             </joint>
             <joint name="Joint_4_Joint">
@@ -35,4 +53,5 @@
                 </state_interface>
                 <state_interface name="velocity"/>
+                <param name="steps_per_radian">${joint4_steps_per_radian}</param>
             </joint>
             <joint name="Joint_5_Joint">
@@ -42,4 +61,5 @@
                 </state_interface>
                 <state_interface name="velocity"/>
+                <param name="steps_per_radian">${joint5_steps_per_radian}</param>
             </joint>
         </ros2_control>

File: src/my_robot_moveit_config/config/armassem1.urdf.xacro (robot description, xacro)
@@ -2,8 +2,16 @@
 <robot xmlns:xacro="http://www.ros.org/wiki/xacro" name="armassem1">
     <xacro:arg name="initial_positions_file" default="initial_positions.yaml" />
+    <xacro:arg name="use_mock_hardware" default="true" />
+    <xacro:arg name="serial_port" default="/dev/ttyACM0" />
+    <xacro:arg name="baud_rate" default="115200" />
     <!-- Import armassem1 urdf file -->
     <xacro:include filename="$(find my_robot_description)/urdf/armassem1.urdf" />
     <!-- Import control_xacro -->
     <xacro:include filename="armassem1.ros2_control.xacro" />
-    <xacro:armassem1_ros2_control name="FakeSystem" initial_positions_file="$(arg initial_positions_file)"/>
+    <xacro:armassem1_ros2_control
+        name="ArmAssem1System"
+        initial_positions_file="$(arg initial_positions_file)"
+        use_mock_hardware="$(arg use_mock_hardware)"
+        serial_port="$(arg serial_port)"
+        baud_rate="$(arg baud_rate)"/>
 </robot>
